File: DemoGit.kicad_sch (KiCad schematic)
At the start: 17 parts, among them J1 USB_B_Micro, J2 Conn_Coaxial, SW1 SW_Push, U1 AP2112K-3.3, U2 RFM95W-915S2, U3 ATSAMD21G15A-A, U4 Waveshare_epaper

Commit message: fix(bom): cambia R2 a 1k
Parts:
- R2: value 10k -> 1k
Changed lines of the file:
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@@
 			)
 		)
-		(property "Value" "10k"
+		(property "Value" "1k"
 			(at 256.54 99.06 90)
 			(show_name no)
@@
 			(at 256.54 102.87 0)
 			(hide yes)
+			(show_name no)
+			(do_not_autoplace no)
+			(effects
+				(font
+					(size 1.27 1.27)
+				)
+			)
+		)
+		(property "Supplier Part Number" ""
+			(at 256.54 102.87 0)
+			(hide yes)
